Commit message: fix gps topic

File: launch/include/config/robot.urdf.xacro (robot description, xacro)
@@ -21,9 +21,9 @@
     <origin xyz="0 0 0" rpy="0 0 0" />
   </joint>
-  <link name="navsat_link"> </link>
+  <link name="gps_link"> </link>
   <joint name="navsat_joint" type="fixed">
     <parent link="chassis_link" />
-    <child link="navsat_link" />
-    <origin xyz="0 0 0" rpy="0 0 0" />
+    <child link="gps_link" />
+    <origin xyz="-0.06222 -0.400 -0.16745" rpy="0 0 0" />
   </joint>
 </robot>

Commit message: add values for imu_link and use gps elevation

File: launch/include/config/robot.urdf.xacro (robot description, xacro)
@@ -13,5 +13,5 @@
     <parent link="chassis_link" />
     <child link="imu_link" />
-    <origin xyz="0 0 0" rpy="0 0 0" />
+    <origin xyz="0.805 0.0 1.3162" rpy="0 0 0" />
   </joint>
   <link name="velodyne"> </link>

Commit message: add angles for velodyne

File: launch/include/config/robot.urdf.xacro (robot description, xacro)
@@ -19,5 +19,5 @@
     <parent link="chassis_link" />
     <child link="velodyne" />
-    <origin xyz="0 0 0" rpy="0 0 0" />
+    <origin xyz="0 0 0" rpy="-0.0035219 0.0256178 -0.0082929" />
   </joint>
   <link name="gps_link"> </link>
